File: hardware/deskcat.kicad_sch (KiCad schematic)
At the start: 24 parts, among them J1 DISP_01_MSP2807, J2 ACCEL_01_ADXL345, J3 ENV_01_BME280, J4 SBC_01_Pi_Zero_W, U1 MCU_01_DevKitC_V4

Commit message: #512: 図は最終配線を描く規則と、回路図の touch 5本を足す
- CONTRIBUTING と hardware/README.md に、図は最終的な配線を描き、測定のためだけの
  一時配線は描かず Wiring-Figure: not-applicable <理由> で通すことを足した。
  図は3つ（breadboard／universal-board／overview）になる前提で、後の2つは #405。
- hardware/deskcat.kicad_sch に touch の5本を足した（DISP-01 の pin 10〜14 を
  LCD-SCLK／TOUCH-CS／LCD-MOSI／LCD-MISO／TOUCH-IRQ へ。MCU に GPIO34 TOUCH-IRQ を追加）。
  注記の「LCD touch pins unused」を EXP-038 の事実に合わせた。
- GPIO34 の header 番号 J2-5 は generate.py の J2 の並びによる。一次資料では未確認。

実機の操作はしていない。KiCad では開いていない。

Refs: #512
Change-Class: review-required
Self-Review: requirements-pass
Self-Review: fresh-context-pass
Self-Review: converged
Instruction-Change: reviewed-as-data
Connections:
- net LCD-MISO: now also J1.13 (T_DO)
- net LCD-MOSI: now also J1.12 (T_DIN)
- net LCD-SCLK: now also J1.10 (T_CLK)
- net TOUCH-CS: now also J1.11 (T_CS)
- new net TOUCH-IRQ: J1.14 (T_IRQ), U1.J2-5 (GPIO34 TOUCH-IRQ)
Other:
- note added: "DeskCat #512 / logical wiring at EXP-019 baseline + EXP-022 UART + EXP-025 LED branches + EXP-038 touch"
- note added: "ENV-01 CSB-J3 bridge: reported soldered, continuity TBD. ACCEL pin numbering: TBD. ACCEL INT1/2 unused. Touch (XPT2046 on DISP-01) 5 wires added at EXP-038; TOUCH-IRQ has no external pull (gpio-assignment.md)."
- note removed: "DeskCat #512 / logical wiring at EXP-019 baseline + EXP-022 UART + EXP-025 LED branches"
- note removed: "ENV-01 CSB-J3 bridge: reported soldered, continuity TBD. ACCEL pin numbering: TBD. LCD touch pins and ACCEL INT1/2 unused."
Changed lines of the file:
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@@
  (generator "eeschema")
  (paper "A1")
- (title_block (title "DeskCat logical wiring #512") (rev "EXP-019 + EXP-022 + EXP-025"))
+ (title_block (title "DeskCat logical wiring #512") (rev "EXP-019 + EXP-022 + EXP-025 + EXP-038"))
 (symbol (lib_id "DeskCat:MCU_01_DevKitC_V4") (at 45 102 0) (unit 1) (in_bom no) (on_board no) (dnp no)
  (property "Reference" "U1" (at 45 71.33 0) (effects (font (size 1.27 1.27))))
@@
  (pin "J3-15")
  (pin "J3-10")
+ (pin "J2-5")
  (instances (project "deskcat" (path "/77da1574-8243-423a-8585-8aedf9ccf9ec" (reference "U1") (unit 1)))))
 (wire (pts (xy 57.7 77.87) (xy 62.78 77.87)) (stroke (width 0) (type default)))
@@
 (wire (pts (xy 57.7 126.13) (xy 62.78 126.13)) (stroke (width 0) (type default)))
 (label "LED-REACT" (at 62.78 126.13 0) (effects (font (size 1.27 1.27))))
+(wire (pts (xy 57.7 128.67) (xy 62.78 128.67)) (stroke (width 0) (type default)))
+(label "TOUCH-IRQ" (at 62.78 128.67 0) (effects (font (size 1.27 1.27))))
 (symbol (lib_id "DeskCat:DISP_01_MSP2807") (at 175 80 0) (unit 1) (in_bom no) (on_board no) (dnp no)
  (property "Reference" "J1" (at 175 63.3 0) (effects (font (size 1.27 1.27))))
@@
  (pin "8")
  (pin "9")
+ (pin "10")
+ (pin "11")
+ (pin "12")
+ (pin "13")
+ (pin "14")
  (instances (project "deskcat" (path "/77da1574-8243-423a-8585-8aedf9ccf9ec" (reference "J1") (unit 1)))))
 (wire (pts (xy 187.7 69.84) (xy 192.78 69.84)) (stroke (width 0) (type default)))
@@
 (wire (pts (xy 187.7 90.16) (xy 192.78 90.16)) (stroke (width 0) (type default)))
 (label "LCD-MISO" (at 192.78 90.16 0) (effects (font (size 1.27 1.27))))
+(wire (pts (xy 187.7 92.7) (xy 192.78 92.7)) (stroke (width 0) (type default)))
+(label "LCD-SCLK" (at 192.78 92.7 0) (effects (font (size 1.27 1.27))))
+(wire (pts (xy 187.7 95.24) (xy 192.78 95.24)) (stroke (width 0) (type default)))
+(label "TOUCH-CS" (at 192.78 95.24 0) (effects (font (size 1.27 1.27))))
+(wire (pts (xy 187.7 97.78) (xy 192.78 97.78)) (stroke (width 0) (type default)))
+(label "LCD-MOSI" (at 192.78 97.78 0) (effects (font (size 1.27 1.27))))
+(wire (pts (xy 187.7 100.32) (xy 192.78 100.32)) (stroke (width 0) (type default)))
+(label "LCD-MISO" (at 192.78 100.32 0) (effects (font (size 1.27 1.27))))
+(wire (pts (xy 187.7 102.86) (xy 192.78 102.86)) (stroke (width 0) (type default)))
+(label "TOUCH-IRQ" (at 192.78 102.86 0) (effects (font (size 1.27 1.27))))
 (symbol (lib_id "DeskCat:ACCEL_01_ADXL345") (at 300 80 0) (unit 1) (in_bom no) (on_board no) (dnp no)
  (property "Reference" "J2" (at 300 64.57 0) (effects (font (size 1.27 1.27))))
@@
 (wire (pts (xy 565 420.81) (xy 565 424.62)) (stroke (width 0) (type default)))
 (label "GND" (at 565 424.62 0) (effects (font (size 1.27 1.27))))
-(text "DeskCat #512 / logical wiring at EXP-019 baseline + EXP-022 UART + EXP-025 LED branches" (at 25 22 0) (effects (font (size 1.5 1.5)) (justify left)))
+(text "DeskCat #512 / logical wiring at EXP-019 baseline + EXP-022 UART + EXP-025 LED branches + EXP-038 touch" (at 25 22 0) (effects (font (size 1.5 1.5)) (justify left)))
 (text "Power sources are separate USB inputs. PROTO-02 physical assembly and final power path: TBD (#405)." (at 25 29 0) (effects (font (size 1.5 1.5)) (justify left)))
 (text "All resistor values: docs/hardware/gpio-assignment.md and led-514-demo.md. KiCad Value fields name the authority." (at 25 444 0) (effects (font (size 1.5 1.5)) (justify left)))
 (text "No component placement or board hole position is implied by this logical schematic. See breadboard/layout.svg." (at 25 452 0) (effects (font (size 1.5 1.5)) (justify left)))
-(text "ENV-01 CSB-J3 bridge: reported soldered, continuity TBD. ACCEL pin numbering: TBD. LCD touch pins and ACCEL INT1/2 unused." (at 25 460 0) (effects (font (size 1.5 1.5)) (justify left)))
+(text "ENV-01 CSB-J3 bridge: reported soldered, continuity TBD. ACCEL pin numbering: TBD. ACCEL INT1/2 unused. Touch (XPT2046 on DISP-01) 5 wires added at EXP-038; TOUCH-IRQ has no external pull (gpio-assignment.md)." (at 25 460 0) (effects (font (size 1.5 1.5)) (justify left)))
 (text "UART series parts are on breadboard; connect signals only while both devices are powered (gpio-assignment.md)." (at 25 468 0) (effects (font (size 1.5 1.5)) (justify left)))
 (text "PROTO-02 is unbuilt. No tested simultaneous UART+LED power-on state is claimed. No servo connected." (at 25 476 0) (effects (font (size 1.5 1.5)) (justify left)))
